File: hardware/v1.1/lensmount-v1.1.sch (KiCad schematic (older format))
At the start: 40 parts, among them J1 VBAT, J10 Picoblade DNP, J2 DETECT, J3 AGND, J4 VDD, J5 DOUT, J6 DIN, J7 DCLK, J8 DGND, J9 USB, P1 TC2030-CTX-Tag-Connect, Q1 2N7002, Q2 2N7002, Q3 2N7002, Q4 AO3401A, Q5 AO3401A, U1 STM32F042F6Px, U2 XC6206PxxxMR, U3 USBLC6-4

Commit message: updated v1.1
Parts:
- removed D1: DNP, Diode_SMD:D_SOD-323F, symbol Device:D_Small
- removed J10: Picoblade DNP, Connector_Molex:Molex_PicoBlade_53398-0571_1x05-1MP_P1.25mm_Vertical, symbol Connector_Generic_MountingPin:Conn_01x05_MountingPin
- added J10: Picoblade DNP, Connector_Molex:Molex_PicoBlade_53398-0471_1x04-1MP_P1.25mm_Vertical, symbol Connector_Generic_MountingPin:Conn_01x04_MountingPin
- J1, J2, J3: Mouser (none) -> 581-709150001025006
- J4, J5, J6, J7, J8: Mouser (none) -> 581-709150001020006
Connections:
- net GND: now also J10.1 (Pin_1), J10.MP (MountPin)
- net VBUS: now also J10.2 (Pin_2)
- net at J1.1 (Pin_1): now also Q4.3 (D)
- net UART_TX: now reaches U1.8 (PA2)
- net UART_TX: now also J10.4 (Pin_4)
- net UART_RX: now reaches U1.9 (PA3)
- net UART_RX: now also J10.3 (Pin_3)
Other:
- note added: "->"
- note added: "<-"
- note added: "Length: 2.0mm"
- note added: "Length: 2.5mm"
Changed lines of the file:
@@
 F 2 "otter:PH-MVF-5365" H 9650 1600 50  0001 C CNN
 F 3 "~" H 9650 1600 50  0001 C CNN
+F 4 "581-709150001025006" H 9650 1600 50  0001 C CNN "Mouser"
 	1    9650 1600
 	1    0    0    -1
@@
 F 2 "otter:PH-MVF-5365" H 9650 2000 50  0001 C CNN
 F 3 "~" H 9650 2000 50  0001 C CNN
+F 4 "581-709150001025006" H 9650 2000 50  0001 C CNN "Mouser"
 	1    9650 2000
 	1    0    0    -1
@@
 F 2 "otter:PH-MVF-5365" H 9650 2200 50  0001 C CNN
 F 3 "~" H 9650 2200 50  0001 C CNN
+F 4 "581-709150001020006" H 9650 2200 50  0001 C CNN "Mouser"
 	1    9650 2200
 	1    0    0    -1
@@
 F 2 "otter:PH-MVF-5365" H 9650 2400 50  0001 C CNN
 F 3 "~" H 9650 2400 50  0001 C CNN
+F 4 "581-709150001020006" H 9650 2400 50  0001 C CNN "Mouser"
 	1    9650 2400
 	1    0    0    -1
@@
 F 2 "otter:PH-MVF-5365" H 9650 2600 50  0001 C CNN
 F 3 "~" H 9650 2600 50  0001 C CNN
+F 4 "581-709150001020006" H 9650 2600 50  0001 C CNN "Mouser"
 	1    9650 2600
 	1    0    0    -1
@@
 F 2 "otter:PH-MVF-5365" H 9650 2800 50  0001 C CNN
 F 3 "~" H 9650 2800 50  0001 C CNN
+F 4 "581-709150001020006" H 9650 2800 50  0001 C CNN "Mouser"
 	1    9650 2800
 	1    0    0    -1
@@
 F 2 "otter:PH-MVF-5365" H 9650 3000 50  0001 C CNN
 F 3 "~" H 9650 3000 50  0001 C CNN
+F 4 "581-709150001020006" H 9650 3000 50  0001 C CNN "Mouser"
 	1    9650 3000
 	1    0    0    -1
@@
 L power:GND #PWR0133
 U 1 1 5F42B46E
-P 9450 4600
-F 0 "#PWR0133" H 9450 4350 50  0001 C CNN
-F 1 "GND" V 9455 4472 50  0000 R CNN
-F 2 "" H 9450 4600 50  0001 C CNN
-F 3 "" H 9450 4600 50  0001 C CNN
-	1    9450 4600
+P 9450 4300
+F 0 "#PWR0133" H 9450 4050 50  0001 C CNN
+F 1 "GND" V 9455 4172 50  0000 R CNN
+F 2 "" H 9450 4300 50  0001 C CNN
+F 3 "" H 9450 4300 50  0001 C CNN
+	1    9450 4300
 	0    1    1    0
-$EndComp
-Text GLabel 9450 4500 0    50   Input ~ 0
-DCLK_5V
-Text GLabel 9450 4400 0    50   Input ~ 0
-DIN_5V
-Text GLabel 9450 4300 0    50   Input ~ 0
-DOUT_5V
-$Comp
-L power:+BATT #PWR0134
-U 1 1 5F42D486
-P 9450 4200
-F 0 "#PWR0134" H 9450 4050 50  0001 C CNN
-F 1 "+BATT" V 9465 4327 50  0000 L CNN
-F 2 "" H 9450 4200 50  0001 C CNN
-F 3 "" H 9450 4200 50  0001 C CNN
-	1    9450 4200
-	0    -1   -1   0
-$EndComp
-$Comp
-L Connector_Generic_MountingPin:Conn_01x05_MountingPin J10
-U 1 1 5F42F74B
-P 9650 4400
-F 0 "J10" H 9738 4364 50  0000 L CNN
-F 1 "Picoblade DNP" H 9738 4273 50  0000 L CNN
-F 2 "Connector_Molex:Molex_PicoBlade_53398-0571_1x05-1MP_P1.25mm_Vertical" H 9650 4400 50  0001 C CNN
-F 3 "~" H 9650 4400 50  0001 C CNN
-	1    9650 4400
-	1    0    0    -1
-$EndComp
-$Comp
-L Device:D_Small D1
-U 1 1 5F43055D
-P 6950 1100
-F 0 "D1" H 6950 1305 50  0000 C CNN
-F 1 "DNP" H 6950 1214 50  0000 C CNN
-F 2 "Diode_SMD:D_SOD-323F" V 6950 1100 50  0001 C CNN
-F 3 "~" V 6950 1100 50  0001 C CNN
-	1    6950 1100
-	1    0    0    -1
-$EndComp
-$Comp
-L power:+BATT #PWR0135
-U 1 1 5F430C9F
-P 7050 1100
-F 0 "#PWR0135" H 7050 950 50  0001 C CNN
-F 1 "+BATT" V 7050 1250 50  0000 L CNN
-F 2 "" H 7050 1100 50  0001 C CNN
-F 3 "" H 7050 1100 50  0001 C CNN
-	1    7050 1100
-	0    1    1    0
-$EndComp
-$Comp
-L power:VBUS #PWR0136
-U 1 1 5F431DE1
-P 6850 1100
-F 0 "#PWR0136" H 6850 950 50  0001 C CNN
-F 1 "VBUS" V 6850 1250 50  0000 L CNN
-F 2 "" H 6850 1100 50  0001 C CNN
-F 3 "" H 6850 1100 50  0001 C CNN
-	1    6850 1100
-	0    -1   -1   0
 $EndComp
 $Comp
@@
 F 2 "otter:PH-MVF-5365" H 9650 1800 50  0001 C CNN
 F 3 "~" H 9650 1800 50  0001 C CNN
+F 4 "581-709150001025006" H 9650 1800 50  0001 C CNN "Mouser"
 	1    9650 1800
 	1    0    0    -1
@@
 Wire Wire Line
 	8450 1950 8450 1900
-Wire Wire Line
-	8700 1600 9450 1600
 $Comp
 L Device:R_Small R12
@@
 Text GLabel 3100 5450 0    50   Input ~ 0
 EN_VBAT
+Wire Notes Line
+	9600 2100 10550 2100
+Wire Notes Line
+	10550 3100 9600 3100
+Wire Notes Line
+	10550 1500 9600 1500
+Wire Notes Line
+	10550 1500 10550 3100
+Text Notes 10600 2600 0    50   ~ 0
+Length: 2.0mm
+Text Notes 10600 1850 0    50   ~ 0
+Length: 2.5mm
+Text GLabel 4300 4950 2    50   Input ~ 0
+UART_TX
+Text GLabel 4300 5050 2    50   Input ~ 0
+UART_RX
+Text Notes 4700 5000 0    50   ~ 0
+->
+Text Notes 4700 5100 0    50   ~ 0
+<-
+Text GLabel 9450 4600 0    50   Input ~ 0
+UART_TX
+Text GLabel 9450 4500 0    50   Input ~ 0
+UART_RX
+$Comp
+L Connector_Generic_MountingPin:Conn_01x04_MountingPin J10
+U 1 1 5F8D18D5
+P 9650 4400
+F 0 "J10" H 9738 4314 50  0000 L CNN
+F 1 "Picoblade DNP" H 9738 4223 50  0000 L CNN
+F 2 "Connector_Molex:Molex_PicoBlade_53398-0471_1x04-1MP_P1.25mm_Vertical" H 9650 4400 50  0001 C CNN
+F 3 "~" H 9650 4400 50  0001 C CNN
+	1    9650 4400
+	1    0    0    -1
+$EndComp
+Wire Wire Line
+	8650 1600 9450 1600
+$Comp
+L power:VBUS #PWR?
+U 1 1 5F959863
+P 9450 4400
+F 0 "#PWR?" H 9450 4250 50  0001 C CNN
+F 1 "VBUS" V 9450 4550 50  0000 L CNN
+F 2 "" H 9450 4400 50  0001 C CNN
+F 3 "" H 9450 4400 50  0001 C CNN
+	1    9450 4400
+	0    -1   -1   0
+$EndComp
 $EndSCHEMATC
