File: hardware/v1.1/lensmount-v1.1.kicad_pcb (KiCad board)
At the start: 2 copper layers, 65 x 65 mm, 41 parts, among them J1 VBAT, J10 Picoblade DNP, J2 DETECT, J3 AGND, J4 VDD, J5 DOUT, J6 DIN, J7 DCLK, J8 DGND, J9 USB, P1 TC2030-CTX-Tag-Connect, Q1 2N7002, Q2 2N7002, Q3 2N7002, Q4 AO3401A, Q5 AO3401A, U1 STM32F042F6Px, U2 XC6206PxxxMR, U3 USBLC6-4

Commit message: updated v1.1
Parts:
- removed D1: DNP, Diode_SMD:D_SOD-323F
- J10: footprint Connector_Molex:Molex_PicoBlade_53398-0571_1x05-1MP_P1.25mm_Vertical -> Connector_Molex:Molex_PicoBlade_53398-0471_1x04-1MP_P1.25mm_Vertical
- Q4, Q5, R10, R11, R12, R13: moved to B.Cu
- moved J10 46.0 mm to (78.7, 89.7), turned to 60 degrees
- moved R11 23.2 mm to (94.0, 124.2), turned to 90 degrees
- moved R12 22.9 mm to (95.8, 124.8), turned to 270 degrees
- moved R13 22.4 mm to (95.4, 126.2), turned to 180 degrees
- moved R10 21.4 mm to (92.2, 126.0)
- moved Q4 20.9 mm to (91.9, 123.8), turned to 90 degrees
- moved Q5 19.6 mm to (98.0, 124.7)
- moved C6 4.10 mm to (90.6, 126.7), turned to 270 degrees
- moved R9 3.15 mm to (91.8, 127.5)
- moved C7 1.20 mm to (97.5, 127.2)
Connections:
- J10 pad 1: +BATT -> GND
- J10 pad 2: DOUT_5V -> VBUS
- J10 pad 3: DIN_5V -> UART_RX
- J10 pad 4: DCLK_5V -> UART_TX
- Q4 pad 3: Net-(Q4-Pad3) -> Net-(J1-Pad1)
- U1 pad 8: Net-(U1-Pad8) -> UART_TX
- U1 pad 9: Net-(U1-Pad9) -> UART_RX
Routing:
- net +BATT: track 52.7 -> 3.47 mm, vias 4 -> 0
- net UART_RX: track 0.00 -> 40.6 mm, vias 0 -> 2
- net UART_TX: track 0.00 -> 39.0 mm, vias 0 -> 2
- net EN_VBUS: track 0.00 -> 18.1 mm, vias 0 -> 2
- net DOUT_5V: track 20.9 -> 3.82 mm, vias 1 -> 0
- net EN_VBAT: track 0.00 -> 14.6 mm, vias 0 -> 2
- net VBUS: track 85.5 -> 99.5 mm
- net DIN_5V: track 16.7 -> 3.80 mm, vias 1 -> 0
- net DETECT: track 0.00 -> 9.20 mm
- net DCLK_5V: track 12.7 -> 5.24 mm
- net NRST: track 12.2 -> 16.1 mm
- net Net-(J4-Pad1): track 0.00 -> 2.64 mm
- net Net-(Q4-Pad1): track 0.00 -> 2.47 mm
- net Net-(Q5-Pad1): track 0.00 -> 2.37 mm
- net Net-(J1-Pad1): track 0.00 -> 1.90 mm
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
Commit message: updated to kicad6
Other:
- net class Default removed
